Commit message: get the ga to run
time to give it some iterations

File: temp0.urdf (robot description, URDF)
Before this commit: robot pepe, 13 links, 12 joints
Links:
- removed link 15
- removed link 19
- removed link 210
- removed link 211
- removed link 212
- removed link 22
- removed link 23
- removed link 24
- removed link 26
- removed link 27
- removed link 28
- link 0: mass 1.5814261342673384 -> 2.3745998898214755; geometry collision cylinder length=1.051961205187508 radius=0.8476575280301925; visual cylinder length=1.051961205187508 radius=0.8476575280301925
- link 11: mass 0.15302195195307494 -> 2.3745998898214755; geometry collision cylinder length=1.051961205187508 radius=0.8476575280301925; visual cylinder length=1.051961205187508 radius=0.8476575280301925
Joints:
- removed joint 15_to_0
- removed joint 19_to_0
- removed joint 210_to_19
- removed joint 211_to_19
- removed joint 212_to_19
- removed joint 22_to_11
- removed joint 23_to_11
- removed joint 24_to_11
- removed joint 26_to_15
- removed joint 27_to_15
- removed joint 28_to_15
- joint 11_to_0: axis 0 1 0 -> 0 0 1; origin xyz=0.3976804631052736 0.6444416384529748 0.13699922461850722 rpy=8.4349774415305 1.5893935971165172 4.864117586330606 -> xyz=0.11866751810199896 0.12529649260884057 0.45253033493619765 rpy=5.041387065644444 4.403987629821016 4.274801344455181

Commit message: let user able to specify a sim_id through cli param

File: temp0.urdf (robot description, URDF)
Before this commit: robot pepe, 2 links, 1 joints
Links:
- added link 22, mass 0.650822219820982; collision cylinder length=0.741830070461249 radius=0.5284501587718825; visual cylinder length=0.741830070461249 radius=0.5284501587718825
- added link 23, mass 0.650822219820982; collision cylinder length=0.741830070461249 radius=0.5284501587718825; visual cylinder length=0.741830070461249 radius=0.5284501587718825
- link 0: mass 2.3745998898214755 -> 0.007320265806382737; geometry collision cylinder length=0.5299822617624999 radius=0.06630676227451326; visual cylinder length=0.5299822617624999 radius=0.06630676227451326
- link 11: mass 2.3745998898214755 -> 0.0005961689949108566; geometry collision cylinder length=0.10278966123950095 radius=0.04296700072513382; visual cylinder length=0.10278966123950095 radius=0.04296700072513382
Joints:
- added joint 22_to_0: type revolute, parent 0, child 22, origin xyz=0.04789953728339402 0.8858095953757255 0.8510448674202954 rpy=10.48488874391538 2.660788820434803 5.755776696955519, axis 0 1 0, limit lower=3.1415 upper=-3.1415 effort=1 velocity=1
- added joint 23_to_0: type revolute, parent 0, child 23, origin xyz=0.04789953728339402 0.8858095953757255 0.8510448674202954 rpy=13.97985165855384 2.660788820434803 5.755776696955519, axis 0 1 0, limit lower=3.1415 upper=-3.1415 effort=1 velocity=1
- joint 11_to_0: origin xyz=0.11866751810199896 0.12529649260884057 0.45253033493619765 rpy=5.041387065644444 4.403987629821016 4.274801344455181 -> xyz=0.3535163972446931 0.9391012838928774 0.2718288971022369 rpy=4.653844063478385 0.7845523927672909 3.172419432061251
