Commit message: let user able to specify a sim_id through cli param

File: test.urdf (robot description, URDF)
Before this commit: robot pepe, 6 links, 5 joints
Links:
- removed link 12
- removed link 13
- removed link 24
- removed link 25
- added link 141, mass 2.371219924663106; collision cylinder length=1.1450995302163955 radius=0.8118753641033697; visual cylinder length=1.1450995302163955 radius=0.8118753641033697
- added link 215, mass 1.6082818338320715; collision cylinder length=0.7085266532788173 radius=0.8500178500145726; visual cylinder length=0.7085266532788173 radius=0.8500178500145726
- added link 22, mass 1.6082818338320715; collision cylinder length=0.7085266532788173 radius=0.8500178500145726; visual cylinder length=0.7085266532788173 radius=0.8500178500145726
- added link 228, mass 1.6082818338320715; collision cylinder length=0.7085266532788173 radius=0.8500178500145726; visual cylinder length=0.7085266532788173 radius=0.8500178500145726
- added link 242, mass 1.6082818338320715; collision cylinder length=0.7085266532788173 radius=0.8500178500145726; visual cylinder length=0.7085266532788173 radius=0.8500178500145726
- added link 255, mass 1.6082818338320715; collision cylinder length=0.7085266532788173 radius=0.8500178500145726; visual cylinder length=0.7085266532788173 radius=0.8500178500145726
- added link 268, mass 1.6082818338320715; collision cylinder length=0.7085266532788173 radius=0.8500178500145726; visual cylinder length=0.7085266532788173 radius=0.8500178500145726
- added link 311, mass 2.927032641435217; collision cylinder length=1.0758014905119015 radius=0.9306208440139438; visual cylinder length=1.0758014905119015 radius=0.9306208440139438
- added link 316, mass 2.927032641435217; collision cylinder length=1.0758014905119015 radius=0.9306208440139438; visual cylinder length=1.0758014905119015 radius=0.9306208440139438
- added link 320, mass 2.927032641435217; collision cylinder length=1.0758014905119015 radius=0.9306208440139438; visual cylinder length=1.0758014905119015 radius=0.9306208440139438
- added link 324, mass 2.927032641435217; collision cylinder length=1.0758014905119015 radius=0.9306208440139438; visual cylinder length=1.0758014905119015 radius=0.9306208440139438
- added link 329, mass 2.927032641435217; collision cylinder length=1.0758014905119015 radius=0.9306208440139438; visual cylinder length=1.0758014905119015 radius=0.9306208440139438
- added link 33, mass 2.927032641435217; collision cylinder length=1.0758014905119015 radius=0.9306208440139438; visual cylinder length=1.0758014905119015 radius=0.9306208440139438
- added link 333, mass 2.927032641435217; collision cylinder length=1.0758014905119015 radius=0.9306208440139438; visual cylinder length=1.0758014905119015 radius=0.9306208440139438
- added link 337, mass 2.927032641435217; collision cylinder length=1.0758014905119015 radius=0.9306208440139438; visual cylinder length=1.0758014905119015 radius=0.9306208440139438
- added link 343, mass 2.927032641435217; collision cylinder length=1.0758014905119015 radius=0.9306208440139438; visual cylinder length=1.0758014905119015 radius=0.9306208440139438
- added link 347, mass 2.927032641435217; collision cylinder length=1.0758014905119015 radius=0.9306208440139438; visual cylinder length=1.0758014905119015 radius=0.9306208440139438
- added link 351, mass 2.927032641435217; collision cylinder length=1.0758014905119015 radius=0.9306208440139438; visual cylinder length=1.0758014905119015 radius=0.9306208440139438
- added link 356, mass 2.927032641435217; collision cylinder length=1.0758014905119015 radius=0.9306208440139438; visual cylinder length=1.0758014905119015 radius=0.9306208440139438
- added link 360, mass 2.927032641435217; collision cylinder length=1.0758014905119015 radius=0.9306208440139438; visual cylinder length=1.0758014905119015 radius=0.9306208440139438
- added link 364, mass 2.927032641435217; collision cylinder length=1.0758014905119015 radius=0.9306208440139438; visual cylinder length=1.0758014905119015 radius=0.9306208440139438
- added link 369, mass 2.927032641435217; collision cylinder length=1.0758014905119015 radius=0.9306208440139438; visual cylinder length=1.0758014905119015 radius=0.9306208440139438
- added link 37, mass 2.927032641435217; collision cylinder length=1.0758014905119015 radius=0.9306208440139438; visual cylinder length=1.0758014905119015 radius=0.9306208440139438
- added link 373, mass 2.927032641435217; collision cylinder length=1.0758014905119015 radius=0.9306208440139438; visual cylinder length=1.0758014905119015 radius=0.9306208440139438
- added link 377, mass 2.927032641435217; collision cylinder length=1.0758014905119015 radius=0.9306208440139438; visual cylinder length=1.0758014905119015 radius=0.9306208440139438
- added link 410, mass 0.3750573152546009; collision cylinder length=0.22633604939576163 radius=0.7262681824986438; visual cylinder length=0.22633604939576163 radius=0.7262681824986438
- added link 412, mass 0.3750573152546009; collision cylinder length=0.22633604939576163 radius=0.7262681824986438; visual cylinder length=0.22633604939576163 radius=0.7262681824986438
- added link 413, mass 0.3750573152546009; collision cylinder length=0.22633604939576163 radius=0.7262681824986438; visual cylinder length=0.22633604939576163 radius=0.7262681824986438
- added link 414, mass 0.3750573152546009; collision cylinder length=0.22633604939576163 radius=0.7262681824986438; visual cylinder length=0.22633604939576163 radius=0.7262681824986438
- added link 417, mass 0.3750573152546009; collision cylinder length=0.22633604939576163 radius=0.7262681824986438; visual cylinder length=0.22633604939576163 radius=0.7262681824986438
- added link 418, mass 0.3750573152546009; collision cylinder length=0.22633604939576163 radius=0.7262681824986438; visual cylinder length=0.22633604939576163 radius=0.7262681824986438
- added link 419, mass 0.3750573152546009; collision cylinder length=0.22633604939576163 radius=0.7262681824986438; visual cylinder length=0.22633604939576163 radius=0.7262681824986438
- added link 421, mass 0.3750573152546009; collision cylinder length=0.22633604939576163 radius=0.7262681824986438; visual cylinder length=0.22633604939576163 radius=0.7262681824986438
- added link 422, mass 0.3750573152546009; collision cylinder length=0.22633604939576163 radius=0.7262681824986438; visual cylinder length=0.22633604939576163 radius=0.7262681824986438
- added link 423, mass 0.3750573152546009; collision cylinder length=0.22633604939576163 radius=0.7262681824986438; visual cylinder length=0.22633604939576163 radius=0.7262681824986438
- added link 425, mass 0.3750573152546009; collision cylinder length=0.22633604939576163 radius=0.7262681824986438; visual cylinder length=0.22633604939576163 radius=0.7262681824986438
- added link 426, mass 0.3750573152546009; collision cylinder length=0.22633604939576163 radius=0.7262681824986438; visual cylinder length=0.22633604939576163 radius=0.7262681824986438
- added link 427, mass 0.3750573152546009; collision cylinder length=0.22633604939576163 radius=0.7262681824986438; visual cylinder length=0.22633604939576163 radius=0.7262681824986438
- added link 430, mass 0.3750573152546009; collision cylinder length=0.22633604939576163 radius=0.7262681824986438; visual cylinder length=0.22633604939576163 radius=0.7262681824986438
- added link 431, mass 0.3750573152546009; collision cylinder length=0.22633604939576163 radius=0.7262681824986438; visual cylinder length=0.22633604939576163 radius=0.7262681824986438
- added link 432, mass 0.3750573152546009; collision cylinder length=0.22633604939576163 radius=0.7262681824986438; visual cylinder length=0.22633604939576163 radius=0.7262681824986438
- added link 434, mass 0.3750573152546009; collision cylinder length=0.22633604939576163 radius=0.7262681824986438; visual cylinder length=0.22633604939576163 radius=0.7262681824986438
- added link 435, mass 0.3750573152546009; collision cylinder length=0.22633604939576163 radius=0.7262681824986438; visual cylinder length=0.22633604939576163 radius=0.7262681824986438
- added link 436, mass 0.3750573152546009; collision cylinder length=0.22633604939576163 radius=0.7262681824986438; visual cylinder length=0.22633604939576163 radius=0.7262681824986438
- added link 438, mass 0.3750573152546009; collision cylinder length=0.22633604939576163 radius=0.7262681824986438; visual cylinder length=0.22633604939576163 radius=0.7262681824986438
- added link 439, mass 0.3750573152546009; collision cylinder length=0.22633604939576163 radius=0.7262681824986438; visual cylinder length=0.22633604939576163 radius=0.7262681824986438
- added link 44, mass 0.3750573152546009; collision cylinder length=0.22633604939576163 radius=0.7262681824986438; visual cylinder length=0.22633604939576163 radius=0.7262681824986438
- added link 440, mass 0.3750573152546009; collision cylinder length=0.22633604939576163 radius=0.7262681824986438; visual cylinder length=0.22633604939576163 radius=0.7262681824986438
- added link 444, mass 0.3750573152546009; collision cylinder length=0.22633604939576163 radius=0.7262681824986438; visual cylinder length=0.22633604939576163 radius=0.7262681824986438
- added link 445, mass 0.3750573152546009; collision cylinder length=0.22633604939576163 radius=0.7262681824986438; visual cylinder length=0.22633604939576163 radius=0.7262681824986438
- added link 446, mass 0.3750573152546009; collision cylinder length=0.22633604939576163 radius=0.7262681824986438; visual cylinder length=0.22633604939576163 radius=0.7262681824986438
- added link 448, mass 0.3750573152546009; collision cylinder length=0.22633604939576163 radius=0.7262681824986438; visual cylinder length=0.22633604939576163 radius=0.7262681824986438
- added link 449, mass 0.3750573152546009; collision cylinder length=0.22633604939576163 radius=0.7262681824986438; visual cylinder length=0.22633604939576163 radius=0.7262681824986438
- added link 45, mass 0.3750573152546009; collision cylinder length=0.22633604939576163 radius=0.7262681824986438; visual cylinder length=0.22633604939576163 radius=0.7262681824986438
- added link 450, mass 0.3750573152546009; collision cylinder length=0.22633604939576163 radius=0.7262681824986438; visual cylinder length=0.22633604939576163 radius=0.7262681824986438
- added link 452, mass 0.3750573152546009; collision cylinder length=0.22633604939576163 radius=0.7262681824986438; visual cylinder length=0.22633604939576163 radius=0.7262681824986438
- added link 453, mass 0.3750573152546009; collision cylinder length=0.22633604939576163 radius=0.7262681824986438; visual cylinder length=0.22633604939576163 radius=0.7262681824986438
- added link 454, mass 0.3750573152546009; collision cylinder length=0.22633604939576163 radius=0.7262681824986438; visual cylinder length=0.22633604939576163 radius=0.7262681824986438
- added link 457, mass 0.3750573152546009; collision cylinder length=0.22633604939576163 radius=0.7262681824986438; visual cylinder length=0.22633604939576163 radius=0.7262681824986438
- added link 458, mass 0.3750573152546009; collision cylinder length=0.22633604939576163 radius=0.7262681824986438; visual cylinder length=0.22633604939576163 radius=0.7262681824986438
- added link 459, mass 0.3750573152546009; collision cylinder length=0.22633604939576163 radius=0.7262681824986438; visual cylinder length=0.22633604939576163 radius=0.7262681824986438
- added link 46, mass 0.3750573152546009; collision cylinder length=0.22633604939576163 radius=0.7262681824986438; visual cylinder length=0.22633604939576163 radius=0.7262681824986438
- added link 461, mass 0.3750573152546009; collision cylinder length=0.22633604939576163 radius=0.7262681824986438; visual cylinder length=0.22633604939576163 radius=0.7262681824986438
- added link 462, mass 0.3750573152546009; collision cylinder length=0.22633604939576163 radius=0.7262681824986438; visual cylinder length=0.22633604939576163 radius=0.7262681824986438
- added link 463, mass 0.3750573152546009; collision cylinder length=0.22633604939576163 radius=0.7262681824986438; visual cylinder length=0.22633604939576163 radius=0.7262681824986438
- added link 465, mass 0.3750573152546009; collision cylinder length=0.22633604939576163 radius=0.7262681824986438; visual cylinder length=0.22633604939576163 radius=0.7262681824986438
- added link 466, mass 0.3750573152546009; collision cylinder length=0.22633604939576163 radius=0.7262681824986438; visual cylinder length=0.22633604939576163 radius=0.7262681824986438
- added link 467, mass 0.3750573152546009; collision cylinder length=0.22633604939576163 radius=0.7262681824986438; visual cylinder length=0.22633604939576163 radius=0.7262681824986438
- added link 470, mass 0.3750573152546009; collision cylinder length=0.22633604939576163 radius=0.7262681824986438; visual cylinder length=0.22633604939576163 radius=0.7262681824986438
- added link 471, mass 0.3750573152546009; collision cylinder length=0.22633604939576163 radius=0.7262681824986438; visual cylinder length=0.22633604939576163 radius=0.7262681824986438
- added link 472, mass 0.3750573152546009; collision cylinder length=0.22633604939576163 radius=0.7262681824986438; visual cylinder length=0.22633604939576163 radius=0.7262681824986438
- added link 474, mass 0.3750573152546009; collision cylinder length=0.22633604939576163 radius=0.7262681824986438; visual cylinder length=0.22633604939576163 radius=0.7262681824986438
- added link 475, mass 0.3750573152546009; collision cylinder length=0.22633604939576163 radius=0.7262681824986438; visual cylinder length=0.22633604939576163 radius=0.7262681824986438
- added link 476, mass 0.3750573152546009; collision cylinder length=0.22633604939576163 radius=0.7262681824986438; visual cylinder length=0.22633604939576163 radius=0.7262681824986438
- added link 478, mass 0.3750573152546009; collision cylinder length=0.22633604939576163 radius=0.7262681824986438; visual cylinder length=0.22633604939576163 radius=0.7262681824986438
- added link 479, mass 0.3750573152546009; collision cylinder length=0.22633604939576163 radius=0.7262681824986438; visual cylinder length=0.22633604939576163 radius=0.7262681824986438
- added link 48, mass 0.3750573152546009; collision cylinder length=0.22633604939576163 radius=0.7262681824986438; visual cylinder length=0.22633604939576163 radius=0.7262681824986438
- added link 480, mass 0.3750573152546009; collision cylinder length=0.22633604939576163 radius=0.7262681824986438; visual cylinder length=0.22633604939576163 radius=0.7262681824986438
- added link 49, mass 0.3750573152546009; collision cylinder length=0.22633604939576163 radius=0.7262681824986438; visual cylinder length=0.22633604939576163 radius=0.7262681824986438
- link 0: mass 1.3749779594994493 -> 0.002296927072579996; geometry collision cylinder length=0.34787170201915224 radius=0.04584469797159296; visual cylinder length=0.34787170201915224 radius=0.04584469797159296
- link 11: mass 1.9999511574405828 -> 2.371219924663106; geometry collision cylinder length=1.1450995302163955 radius=0.8118753641033697; visual cylinder length=1.1450995302163955 radius=0.8118753641033697
Joints:
- removed joint 12_to_0
- removed joint 13_to_0
- removed joint 24_to_0
- removed joint 25_to_0
- added joint 141_to_0: type revolute, parent 0, child 141, origin xyz=0.3487552547759922 0.4287697536007756 0.3870244515537885 rpy=9.399597536942023 5.646478324597923 2.9029606919443376, axis 0 0 1, limit lower=3.1415 upper=-3.1415 effort=1 velocity=1
- added joint 215_to_11: type revolute, parent 11, child 215, origin xyz=0.8704126844852472 0.15505226027397123 0.73850089972101 rpy=3.410601012829197 5.616259286488804 5.792622980579965, axis 0 0 1, limit lower=3.1415 upper=-3.1415 effort=1 velocity=1
- added joint 228_to_11: type revolute, parent 11, child 228, origin xyz=0.8704126844852472 0.15505226027397123 0.73850089972101 rpy=4.547468017105596 5.616259286488804 5.792622980579965, axis 0 0 1, limit lower=3.1415 upper=-3.1415 effort=1 velocity=1
- added joint 22_to_11: type revolute, parent 11, child 22, origin xyz=0.8704126844852472 0.15505226027397123 0.73850089972101 rpy=2.273734008552798 5.616259286488804 5.792622980579965, axis 0 0 1, limit lower=3.1415 upper=-3.1415 effort=1 velocity=1
- added joint 242_to_141: type revolute, parent 141, child 242, origin xyz=0.8704126844852472 0.15505226027397123 0.73850089972101 rpy=2.273734008552798 5.616259286488804 5.792622980579965, axis 0 0 1, limit lower=3.1415 upper=-3.1415 effort=1 velocity=1
- added joint 255_to_141: type revolute, parent 141, child 255, origin xyz=0.8704126844852472 0.15505226027397123 0.73850089972101 rpy=3.410601012829197 5.616259286488804 5.792622980579965, axis 0 0 1, limit lower=3.1415 upper=-3.1415 effort=1 velocity=1
- added joint 268_to_141: type revolute, parent 141, child 268, origin xyz=0.8704126844852472 0.15505226027397123 0.73850089972101 rpy=4.547468017105596 5.616259286488804 5.792622980579965, axis 0 0 1, limit lower=3.1415 upper=-3.1415 effort=1 velocity=1
- added joint 311_to_22: type revolute, parent 22, child 311, origin xyz=0.9999 0.39674765931556455 0.9005141757063853 rpy=3.8248939579930674 0.9151792664694063 6.282556988648868, axis 0 1 0, limit lower=3.1415 upper=-3.1415 effort=1 velocity=1
- added joint 316_to_215: type revolute, parent 215, child 316, origin xyz=0.9999 0.39674765931556455 0.9005141757063853 rpy=1.9124469789965337 0.9151792664694063 6.282556988648868, axis 0 1 0, limit lower=3.1415 upper=-3.1415 effort=1 velocity=1
- added joint 320_to_215: type revolute, parent 215, child 320, origin xyz=0.9999 0.39674765931556455 0.9005141757063853 rpy=2.8686704684948006 0.9151792664694063 6.282556988648868, axis 0 1 0, limit lower=3.1415 upper=-3.1415 effort=1 velocity=1
- added joint 324_to_215: type revolute, parent 215, child 324, origin xyz=0.9999 0.39674765931556455 0.9005141757063853 rpy=3.8248939579930674 0.9151792664694063 6.282556988648868, axis 0 1 0, limit lower=3.1415 upper=-3.1415 effort=1 velocity=1
- added joint 329_to_228: type revolute, parent 228, child 329, origin xyz=0.9999 0.39674765931556455 0.9005141757063853 rpy=1.9124469789965337 0.9151792664694063 6.282556988648868, axis 0 1 0, limit lower=3.1415 upper=-3.1415 effort=1 velocity=1
- added joint 333_to_228: type revolute, parent 228, child 333, origin xyz=0.9999 0.39674765931556455 0.9005141757063853 rpy=2.8686704684948006 0.9151792664694063 6.282556988648868, axis 0 1 0, limit lower=3.1415 upper=-3.1415 effort=1 velocity=1
- added joint 337_to_228: type revolute, parent 228, child 337, origin xyz=0.9999 0.39674765931556455 0.9005141757063853 rpy=3.8248939579930674 0.9151792664694063 6.282556988648868, axis 0 1 0, limit lower=3.1415 upper=-3.1415 effort=1 velocity=1
- added joint 33_to_22: type revolute, parent 22, child 33, origin xyz=0.9999 0.39674765931556455 0.9005141757063853 rpy=1.9124469789965337 0.9151792664694063 6.282556988648868, axis 0 1 0, limit lower=3.1415 upper=-3.1415 effort=1 velocity=1
- added joint 343_to_242: type revolute, parent 242, child 343, origin xyz=0.9999 0.39674765931556455 0.9005141757063853 rpy=1.9124469789965337 0.9151792664694063 6.282556988648868, axis 0 1 0, limit lower=3.1415 upper=-3.1415 effort=1 velocity=1
- added joint 347_to_242: type revolute, parent 242, child 347, origin xyz=0.9999 0.39674765931556455 0.9005141757063853 rpy=2.8686704684948006 0.9151792664694063 6.282556988648868, axis 0 1 0, limit lower=3.1415 upper=-3.1415 effort=1 velocity=1
- added joint 351_to_242: type revolute, parent 242, child 351, origin xyz=0.9999 0.39674765931556455 0.9005141757063853 rpy=3.8248939579930674 0.9151792664694063 6.282556988648868, axis 0 1 0, limit lower=3.1415 upper=-3.1415 effort=1 velocity=1
- added joint 356_to_255: type revolute, parent 255, child 356, origin xyz=0.9999 0.39674765931556455 0.9005141757063853 rpy=1.9124469789965337 0.9151792664694063 6.282556988648868, axis 0 1 0, limit lower=3.1415 upper=-3.1415 effort=1 velocity=1
- added joint 360_to_255: type revolute, parent 255, child 360, origin xyz=0.9999 0.39674765931556455 0.9005141757063853 rpy=2.8686704684948006 0.9151792664694063 6.282556988648868, axis 0 1 0, limit lower=3.1415 upper=-3.1415 effort=1 velocity=1
- added joint 364_to_255: type revolute, parent 255, child 364, origin xyz=0.9999 0.39674765931556455 0.9005141757063853 rpy=3.8248939579930674 0.9151792664694063 6.282556988648868, axis 0 1 0, limit lower=3.1415 upper=-3.1415 effort=1 velocity=1
- added joint 369_to_268: type revolute, parent 268, child 369, origin xyz=0.9999 0.39674765931556455 0.9005141757063853 rpy=1.9124469789965337 0.9151792664694063 6.282556988648868, axis 0 1 0, limit lower=3.1415 upper=-3.1415 effort=1 velocity=1
- added joint 373_to_268: type revolute, parent 268, child 373, origin xyz=0.9999 0.39674765931556455 0.9005141757063853 rpy=2.8686704684948006 0.9151792664694063 6.282556988648868, axis 0 1 0, limit lower=3.1415 upper=-3.1415 effort=1 velocity=1
- added joint 377_to_268: type revolute, parent 268, child 377, origin xyz=0.9999 0.39674765931556455 0.9005141757063853 rpy=3.8248939579930674 0.9151792664694063 6.282556988648868, axis 0 1 0, limit lower=3.1415 upper=-3.1415 effort=1 velocity=1
- added joint 37_to_22: type revolute, parent 22, child 37, origin xyz=0.9999 0.39674765931556455 0.9005141757063853 rpy=2.8686704684948006 0.9151792664694063 6.282556988648868, axis 0 1 0, limit lower=3.1415 upper=-3.1415 effort=1 velocity=1
- added joint 410_to_37: type revolute, parent 37, child 410, origin xyz=0.3515571687244322 0.6192887848937129 0.5941360090781349 rpy=4.625458558909664 5.991712807238684 1.0105649285686076, axis 1 0 0, limit lower=3.1415 upper=-3.1415 effort=1 velocity=1
- added joint 412_to_311: type revolute, parent 311, child 412, origin xyz=0.3515571687244322 0.6192887848937129 0.5941360090781349 rpy=2.312729279454832 5.991712807238684 1.0105649285686076, axis 1 0 0, limit lower=3.1415 upper=-3.1415 effort=1 velocity=1
- added joint 413_to_311: type revolute, parent 311, child 413, origin xyz=0.3515571687244322 0.6192887848937129 0.5941360090781349 rpy=3.4690939191822485 5.991712807238684 1.0105649285686076, axis 1 0 0, limit lower=3.1415 upper=-3.1415 effort=1 velocity=1
- added joint 414_to_311: type revolute, parent 311, child 414, origin xyz=0.3515571687244322 0.6192887848937129 0.5941360090781349 rpy=4.625458558909664 5.991712807238684 1.0105649285686076, axis 1 0 0, limit lower=3.1415 upper=-3.1415 effort=1 velocity=1
- added joint 417_to_316: type revolute, parent 316, child 417, origin xyz=0.3515571687244322 0.6192887848937129 0.5941360090781349 rpy=2.312729279454832 5.991712807238684 1.0105649285686076, axis 1 0 0, limit lower=3.1415 upper=-3.1415 effort=1 velocity=1
- added joint 418_to_316: type revolute, parent 316, child 418, origin xyz=0.3515571687244322 0.6192887848937129 0.5941360090781349 rpy=3.4690939191822485 5.991712807238684 1.0105649285686076, axis 1 0 0, limit lower=3.1415 upper=-3.1415 effort=1 velocity=1
- added joint 419_to_316: type revolute, parent 316, child 419, origin xyz=0.3515571687244322 0.6192887848937129 0.5941360090781349 rpy=4.625458558909664 5.991712807238684 1.0105649285686076, axis 1 0 0, limit lower=3.1415 upper=-3.1415 effort=1 velocity=1
- added joint 421_to_320: type revolute, parent 320, child 421, origin xyz=0.3515571687244322 0.6192887848937129 0.5941360090781349 rpy=2.312729279454832 5.991712807238684 1.0105649285686076, axis 1 0 0, limit lower=3.1415 upper=-3.1415 effort=1 velocity=1
- added joint 422_to_320: type revolute, parent 320, child 422, origin xyz=0.3515571687244322 0.6192887848937129 0.5941360090781349 rpy=3.4690939191822485 5.991712807238684 1.0105649285686076, axis 1 0 0, limit lower=3.1415 upper=-3.1415 effort=1 velocity=1
- added joint 423_to_320: type revolute, parent 320, child 423, origin xyz=0.3515571687244322 0.6192887848937129 0.5941360090781349 rpy=4.625458558909664 5.991712807238684 1.0105649285686076, axis 1 0 0, limit lower=3.1415 upper=-3.1415 effort=1 velocity=1
- added joint 425_to_324: type revolute, parent 324, child 425, origin xyz=0.3515571687244322 0.6192887848937129 0.5941360090781349 rpy=2.312729279454832 5.991712807238684 1.0105649285686076, axis 1 0 0, limit lower=3.1415 upper=-3.1415 effort=1 velocity=1
- added joint 426_to_324: type revolute, parent 324, child 426, origin xyz=0.3515571687244322 0.6192887848937129 0.5941360090781349 rpy=3.4690939191822485 5.991712807238684 1.0105649285686076, axis 1 0 0, limit lower=3.1415 upper=-3.1415 effort=1 velocity=1
- added joint 427_to_324: type revolute, parent 324, child 427, origin xyz=0.3515571687244322 0.6192887848937129 0.5941360090781349 rpy=4.625458558909664 5.991712807238684 1.0105649285686076, axis 1 0 0, limit lower=3.1415 upper=-3.1415 effort=1 velocity=1
- added joint 430_to_329: type revolute, parent 329, child 430, origin xyz=0.3515571687244322 0.6192887848937129 0.5941360090781349 rpy=2.312729279454832 5.991712807238684 1.0105649285686076, axis 1 0 0, limit lower=3.1415 upper=-3.1415 effort=1 velocity=1
- added joint 431_to_329: type revolute, parent 329, child 431, origin xyz=0.3515571687244322 0.6192887848937129 0.5941360090781349 rpy=3.4690939191822485 5.991712807238684 1.0105649285686076, axis 1 0 0, limit lower=3.1415 upper=-3.1415 effort=1 velocity=1
- added joint 432_to_329: type revolute, parent 329, child 432, origin xyz=0.3515571687244322 0.6192887848937129 0.5941360090781349 rpy=4.625458558909664 5.991712807238684 1.0105649285686076, axis 1 0 0, limit lower=3.1415 upper=-3.1415 effort=1 velocity=1
- added joint 434_to_333: type revolute, parent 333, child 434, origin xyz=0.3515571687244322 0.6192887848937129 0.5941360090781349 rpy=2.312729279454832 5.991712807238684 1.0105649285686076, axis 1 0 0, limit lower=3.1415 upper=-3.1415 effort=1 velocity=1
- added joint 435_to_333: type revolute, parent 333, child 435, origin xyz=0.3515571687244322 0.6192887848937129 0.5941360090781349 rpy=3.4690939191822485 5.991712807238684 1.0105649285686076, axis 1 0 0, limit lower=3.1415 upper=-3.1415 effort=1 velocity=1
- added joint 436_to_333: type revolute, parent 333, child 436, origin xyz=0.3515571687244322 0.6192887848937129 0.5941360090781349 rpy=4.625458558909664 5.991712807238684 1.0105649285686076, axis 1 0 0, limit lower=3.1415 upper=-3.1415 effort=1 velocity=1
- added joint 438_to_337: type revolute, parent 337, child 438, origin xyz=0.3515571687244322 0.6192887848937129 0.5941360090781349 rpy=2.312729279454832 5.991712807238684 1.0105649285686076, axis 1 0 0, limit lower=3.1415 upper=-3.1415 effort=1 velocity=1
- added joint 439_to_337: type revolute, parent 337, child 439, origin xyz=0.3515571687244322 0.6192887848937129 0.5941360090781349 rpy=3.4690939191822485 5.991712807238684 1.0105649285686076, axis 1 0 0, limit lower=3.1415 upper=-3.1415 effort=1 velocity=1
- added joint 440_to_337: type revolute, parent 337, child 440, origin xyz=0.3515571687244322 0.6192887848937129 0.5941360090781349 rpy=4.625458558909664 5.991712807238684 1.0105649285686076, axis 1 0 0, limit lower=3.1415 upper=-3.1415 effort=1 velocity=1
- added joint 444_to_343: type revolute, parent 343, child 444, origin xyz=0.3515571687244322 0.6192887848937129 0.5941360090781349 rpy=2.312729279454832 5.991712807238684 1.0105649285686076, axis 1 0 0, limit lower=3.1415 upper=-3.1415 effort=1 velocity=1
- added joint 445_to_343: type revolute, parent 343, child 445, origin xyz=0.3515571687244322 0.6192887848937129 0.5941360090781349 rpy=3.4690939191822485 5.991712807238684 1.0105649285686076, axis 1 0 0, limit lower=3.1415 upper=-3.1415 effort=1 velocity=1
- added joint 446_to_343: type revolute, parent 343, child 446, origin xyz=0.3515571687244322 0.6192887848937129 0.5941360090781349 rpy=4.625458558909664 5.991712807238684 1.0105649285686076, axis 1 0 0, limit lower=3.1415 upper=-3.1415 effort=1 velocity=1
- added joint 448_to_347: type revolute, parent 347, child 448, origin xyz=0.3515571687244322 0.6192887848937129 0.5941360090781349 rpy=2.312729279454832 5.991712807238684 1.0105649285686076, axis 1 0 0, limit lower=3.1415 upper=-3.1415 effort=1 velocity=1
- added joint 449_to_347: type revolute, parent 347, child 449, origin xyz=0.3515571687244322 0.6192887848937129 0.5941360090781349 rpy=3.4690939191822485 5.991712807238684 1.0105649285686076, axis 1 0 0, limit lower=3.1415 upper=-3.1415 effort=1 velocity=1
- added joint 44_to_33: type revolute, parent 33, child 44, origin xyz=0.3515571687244322 0.6192887848937129 0.5941360090781349 rpy=2.312729279454832 5.991712807238684 1.0105649285686076, axis 1 0 0, limit lower=3.1415 upper=-3.1415 effort=1 velocity=1
- added joint 450_to_347: type revolute, parent 347, child 450, origin xyz=0.3515571687244322 0.6192887848937129 0.5941360090781349 rpy=4.625458558909664 5.991712807238684 1.0105649285686076, axis 1 0 0, limit lower=3.1415 upper=-3.1415 effort=1 velocity=1
- added joint 452_to_351: type revolute, parent 351, child 452, origin xyz=0.3515571687244322 0.6192887848937129 0.5941360090781349 rpy=2.312729279454832 5.991712807238684 1.0105649285686076, axis 1 0 0, limit lower=3.1415 upper=-3.1415 effort=1 velocity=1
- added joint 453_to_351: type revolute, parent 351, child 453, origin xyz=0.3515571687244322 0.6192887848937129 0.5941360090781349 rpy=3.4690939191822485 5.991712807238684 1.0105649285686076, axis 1 0 0, limit lower=3.1415 upper=-3.1415 effort=1 velocity=1
- added joint 454_to_351: type revolute, parent 351, child 454, origin xyz=0.3515571687244322 0.6192887848937129 0.5941360090781349 rpy=4.625458558909664 5.991712807238684 1.0105649285686076, axis 1 0 0, limit lower=3.1415 upper=-3.1415 effort=1 velocity=1
- added joint 457_to_356: type revolute, parent 356, child 457, origin xyz=0.3515571687244322 0.6192887848937129 0.5941360090781349 rpy=2.312729279454832 5.991712807238684 1.0105649285686076, axis 1 0 0, limit lower=3.1415 upper=-3.1415 effort=1 velocity=1
- added joint 458_to_356: type revolute, parent 356, child 458, origin xyz=0.3515571687244322 0.6192887848937129 0.5941360090781349 rpy=3.4690939191822485 5.991712807238684 1.0105649285686076, axis 1 0 0, limit lower=3.1415 upper=-3.1415 effort=1 velocity=1
- added joint 459_to_356: type revolute, parent 356, child 459, origin xyz=0.3515571687244322 0.6192887848937129 0.5941360090781349 rpy=4.625458558909664 5.991712807238684 1.0105649285686076, axis 1 0 0, limit lower=3.1415 upper=-3.1415 effort=1 velocity=1
- added joint 45_to_33: type revolute, parent 33, child 45, origin xyz=0.3515571687244322 0.6192887848937129 0.5941360090781349 rpy=3.4690939191822485 5.991712807238684 1.0105649285686076, axis 1 0 0, limit lower=3.1415 upper=-3.1415 effort=1 velocity=1
- added joint 461_to_360: type revolute, parent 360, child 461, origin xyz=0.3515571687244322 0.6192887848937129 0.5941360090781349 rpy=2.312729279454832 5.991712807238684 1.0105649285686076, axis 1 0 0, limit lower=3.1415 upper=-3.1415 effort=1 velocity=1
- added joint 462_to_360: type revolute, parent 360, child 462, origin xyz=0.3515571687244322 0.6192887848937129 0.5941360090781349 rpy=3.4690939191822485 5.991712807238684 1.0105649285686076, axis 1 0 0, limit lower=3.1415 upper=-3.1415 effort=1 velocity=1
- added joint 463_to_360: type revolute, parent 360, child 463, origin xyz=0.3515571687244322 0.6192887848937129 0.5941360090781349 rpy=4.625458558909664 5.991712807238684 1.0105649285686076, axis 1 0 0, limit lower=3.1415 upper=-3.1415 effort=1 velocity=1
- added joint 465_to_364: type revolute, parent 364, child 465, origin xyz=0.3515571687244322 0.6192887848937129 0.5941360090781349 rpy=2.312729279454832 5.991712807238684 1.0105649285686076, axis 1 0 0, limit lower=3.1415 upper=-3.1415 effort=1 velocity=1
- added joint 466_to_364: type revolute, parent 364, child 466, origin xyz=0.3515571687244322 0.6192887848937129 0.5941360090781349 rpy=3.4690939191822485 5.991712807238684 1.0105649285686076, axis 1 0 0, limit lower=3.1415 upper=-3.1415 effort=1 velocity=1
- added joint 467_to_364: type revolute, parent 364, child 467, origin xyz=0.3515571687244322 0.6192887848937129 0.5941360090781349 rpy=4.625458558909664 5.991712807238684 1.0105649285686076, axis 1 0 0, limit lower=3.1415 upper=-3.1415 effort=1 velocity=1
- added joint 46_to_33: type revolute, parent 33, child 46, origin xyz=0.3515571687244322 0.6192887848937129 0.5941360090781349 rpy=4.625458558909664 5.991712807238684 1.0105649285686076, axis 1 0 0, limit lower=3.1415 upper=-3.1415 effort=1 velocity=1
- added joint 470_to_369: type revolute, parent 369, child 470, origin xyz=0.3515571687244322 0.6192887848937129 0.5941360090781349 rpy=2.312729279454832 5.991712807238684 1.0105649285686076, axis 1 0 0, limit lower=3.1415 upper=-3.1415 effort=1 velocity=1
- added joint 471_to_369: type revolute, parent 369, child 471, origin xyz=0.3515571687244322 0.6192887848937129 0.5941360090781349 rpy=3.4690939191822485 5.991712807238684 1.0105649285686076, axis 1 0 0, limit lower=3.1415 upper=-3.1415 effort=1 velocity=1
- added joint 472_to_369: type revolute, parent 369, child 472, origin xyz=0.3515571687244322 0.6192887848937129 0.5941360090781349 rpy=4.625458558909664 5.991712807238684 1.0105649285686076, axis 1 0 0, limit lower=3.1415 upper=-3.1415 effort=1 velocity=1
- added joint 474_to_373: type revolute, parent 373, child 474, origin xyz=0.3515571687244322 0.6192887848937129 0.5941360090781349 rpy=2.312729279454832 5.991712807238684 1.0105649285686076, axis 1 0 0, limit lower=3.1415 upper=-3.1415 effort=1 velocity=1
- added joint 475_to_373: type revolute, parent 373, child 475, origin xyz=0.3515571687244322 0.6192887848937129 0.5941360090781349 rpy=3.4690939191822485 5.991712807238684 1.0105649285686076, axis 1 0 0, limit lower=3.1415 upper=-3.1415 effort=1 velocity=1
- added joint 476_to_373: type revolute, parent 373, child 476, origin xyz=0.3515571687244322 0.6192887848937129 0.5941360090781349 rpy=4.625458558909664 5.991712807238684 1.0105649285686076, axis 1 0 0, limit lower=3.1415 upper=-3.1415 effort=1 velocity=1
- added joint 478_to_377: type revolute, parent 377, child 478, origin xyz=0.3515571687244322 0.6192887848937129 0.5941360090781349 rpy=2.312729279454832 5.991712807238684 1.0105649285686076, axis 1 0 0, limit lower=3.1415 upper=-3.1415 effort=1 velocity=1
- added joint 479_to_377: type revolute, parent 377, child 479, origin xyz=0.3515571687244322 0.6192887848937129 0.5941360090781349 rpy=3.4690939191822485 5.991712807238684 1.0105649285686076, axis 1 0 0, limit lower=3.1415 upper=-3.1415 effort=1 velocity=1
- added joint 480_to_377: type revolute, parent 377, child 480, origin xyz=0.3515571687244322 0.6192887848937129 0.5941360090781349 rpy=4.625458558909664 5.991712807238684 1.0105649285686076, axis 1 0 0, limit lower=3.1415 upper=-3.1415 effort=1 velocity=1
- added joint 48_to_37: type revolute, parent 37, child 48, origin xyz=0.3515571687244322 0.6192887848937129 0.5941360090781349 rpy=2.312729279454832 5.991712807238684 1.0105649285686076, axis 1 0 0, limit lower=3.1415 upper=-3.1415 effort=1 velocity=1
- added joint 49_to_37: type revolute, parent 37, child 49, origin xyz=0.3515571687244322 0.6192887848937129 0.5941360090781349 rpy=3.4690939191822485 5.991712807238684 1.0105649285686076, axis 1 0 0, limit lower=3.1415 upper=-3.1415 effort=1 velocity=1
- joint 11_to_0: origin xyz=0.005471728189169411 0.8221972834451906 0.6927316773471869 rpy=1.645880349662696 4.079545910415286 3.726384375929282 -> xyz=0.3487552547759922 0.4287697536007756 0.3870244515537885 rpy=6.266398357961349 5.646478324597923 2.9029606919443376
