Commit message: add ability to change sim mode in run_ga by cli argument

File: temp0.urdf (robot description, URDF)
Before this commit: robot pepe, 4 links, 3 joints
Links:
- removed link 23
- added link 13, mass 4.264862617044469; collision cylinder length=1.6167235865337606 radius=0.9163464452434805; visual cylinder length=1.6167235865337606 radius=0.9163464452434805
- added link 15, mass 4.264862617044469; collision cylinder length=1.6167235865337606 radius=0.9163464452434805; visual cylinder length=1.6167235865337606 radius=0.9163464452434805
- added link 24, mass 1.148510144550484; collision cylinder length=0.9702427187033971 radius=0.6138359013033038; visual cylinder length=0.9702427187033971 radius=0.6138359013033038
- added link 26, mass 1.148510144550484; collision cylinder length=0.9702427187033971 radius=0.6138359013033038; visual cylinder length=0.9702427187033971 radius=0.6138359013033038
- link 0: mass 0.007320265806382737 -> 0.2993427185894939; geometry collision cylinder length=0.35089437110595445 radius=0.5211001667870432; visual cylinder length=0.35089437110595445 radius=0.5211001667870432
- link 11: mass 0.0005961689949108566 -> 4.264862617044469; geometry collision cylinder length=1.6167235865337606 radius=0.9163464452434805; visual cylinder length=1.6167235865337606 radius=0.9163464452434805
- link 22: mass 0.650822219820982 -> 1.148510144550484; geometry collision cylinder length=0.9702427187033971 radius=0.6138359013033038; visual cylinder length=0.9702427187033971 radius=0.6138359013033038
Joints:
- removed joint 22_to_0
- removed joint 23_to_0
- added joint 13_to_0: type revolute, parent 0, child 13, origin xyz=0.30953915295501044 0.6895189303275684 0.5495245631995184 rpy=15.925258267913355 0.7206710599815701 6.282556988648868, axis 1 0 0, limit lower=3.1415 upper=-3.1415 effort=1 velocity=1
- added joint 15_to_0: type revolute, parent 0, child 15, origin xyz=0.30953915295501044 0.6895189303275684 0.5495245631995184 rpy=21.23367769055114 0.7206710599815701 6.282556988648868, axis 1 0 0, limit lower=3.1415 upper=-3.1415 effort=1 velocity=1
- added joint 22_to_11: type revolute, parent 11, child 22, origin xyz=0.25439540509300496 0.2289664483963053 0.13768350084241276 rpy=12.253927186812717 1.437516484625504 4.5765889171154335, axis 0 1 0, limit lower=3.1415 upper=-3.1415 effort=1 velocity=1
- added joint 24_to_13: type revolute, parent 13, child 24, origin xyz=0.25439540509300496 0.2289664483963053 0.13768350084241276 rpy=12.253927186812717 1.437516484625504 4.5765889171154335, axis 0 1 0, limit lower=3.1415 upper=-3.1415 effort=1 velocity=1
- added joint 26_to_15: type revolute, parent 15, child 26, origin xyz=0.25439540509300496 0.2289664483963053 0.13768350084241276 rpy=12.253927186812717 1.437516484625504 4.5765889171154335, axis 0 1 0, limit lower=3.1415 upper=-3.1415 effort=1 velocity=1
- joint 11_to_0: axis 0 0 1 -> 1 0 0; origin xyz=0.3535163972446931 0.9391012838928774 0.2718288971022369 rpy=4.653844063478385 0.7845523927672909 3.172419432061251 -> xyz=0.30953915295501044 0.6895189303275684 0.5495245631995184 rpy=10.61683884527557 0.7206710599815701 6.282556988648868

File: test.urdf (robot description, URDF)
Before this commit: robot pepe, 81 links, 80 joints
Links:
- removed link 141
- removed link 215
- removed link 228
- removed link 242
- removed link 255
- removed link 268
- removed link 311
- removed link 316
- removed link 320
- removed link 324
- removed link 329
- removed link 33
- removed link 333
- removed link 337
- removed link 343
- removed link 347
- removed link 351
- removed link 356
- removed link 360
- removed link 364
- removed link 369
- removed link 37
- removed link 373
- removed link 377
- removed link 410
- removed link 412
- removed link 413
- removed link 414
- removed link 417
- removed link 418
- removed link 419
- removed link 421
- removed link 422
- removed link 423
- removed link 425
- removed link 426
- removed link 427
- removed link 430
- removed link 431
- removed link 432
- removed link 434
- removed link 435
- removed link 436
- removed link 438
- removed link 439
- removed link 44
- removed link 440
- removed link 444
- removed link 445
- removed link 446
- removed link 448
- removed link 449
- removed link 45
- removed link 450
- removed link 452
- removed link 453
- removed link 454
- removed link 457
- removed link 458
- removed link 459
- removed link 46
- removed link 461
- removed link 462
- removed link 463
- removed link 465
- removed link 466
- removed link 467
- removed link 470
- removed link 471
- removed link 472
- removed link 474
- removed link 475
- removed link 476
- removed link 478
- removed link 479
- removed link 48
- removed link 480
- removed link 49
- added link 23, mass 0.01063960190458224; collision cylinder length=0.457697418014013 radius=0.08601981846400453; visual cylinder length=0.457697418014013 radius=0.08601981846400453
- link 0: mass 0.002296927072579996 -> 0.01063960190458224; geometry collision cylinder length=0.457697418014013 radius=0.08601981846400453; visual cylinder length=0.457697418014013 radius=0.08601981846400453
- link 11: mass 2.371219924663106 -> 1.219129850958162; geometry collision cylinder length=1.447742967353149 radius=0.5177311722190563; visual cylinder length=1.447742967353149 radius=0.5177311722190563
- link 22: mass 1.6082818338320715 -> 0.01063960190458224; geometry collision cylinder length=0.457697418014013 radius=0.08601981846400453; visual cylinder length=0.457697418014013 radius=0.08601981846400453
Joints:
- removed joint 141_to_0
- removed joint 215_to_11
- removed joint 228_to_11
- removed joint 242_to_141
- removed joint 255_to_141
- removed joint 268_to_141
- removed joint 311_to_22
- removed joint 316_to_215
- removed joint 320_to_215
- removed joint 324_to_215
- removed joint 329_to_228
- removed joint 333_to_228
- removed joint 337_to_228
- removed joint 33_to_22
- removed joint 343_to_242
- removed joint 347_to_242
- removed joint 351_to_242
- removed joint 356_to_255
- removed joint 360_to_255
- removed joint 364_to_255
- removed joint 369_to_268
- removed joint 373_to_268
- removed joint 377_to_268
- removed joint 37_to_22
- removed joint 410_to_37
- removed joint 412_to_311
- removed joint 413_to_311
- removed joint 414_to_311
- removed joint 417_to_316
- removed joint 418_to_316
- removed joint 419_to_316
- removed joint 421_to_320
- removed joint 422_to_320
- removed joint 423_to_320
- removed joint 425_to_324
- removed joint 426_to_324
- removed joint 427_to_324
- removed joint 430_to_329
- removed joint 431_to_329
- removed joint 432_to_329
- removed joint 434_to_333
- removed joint 435_to_333
- removed joint 436_to_333
- removed joint 438_to_337
- removed joint 439_to_337
- removed joint 440_to_337
- removed joint 444_to_343
- removed joint 445_to_343
- removed joint 446_to_343
- removed joint 448_to_347
- removed joint 449_to_347
- removed joint 44_to_33
- removed joint 450_to_347
- removed joint 452_to_351
- removed joint 453_to_351
- removed joint 454_to_351
- removed joint 457_to_356
- removed joint 458_to_356
- removed joint 459_to_356
- removed joint 45_to_33
- removed joint 461_to_360
- removed joint 462_to_360
- removed joint 463_to_360
- removed joint 465_to_364
- removed joint 466_to_364
- removed joint 467_to_364
- removed joint 46_to_33
- removed joint 470_to_369
- removed joint 471_to_369
- removed joint 472_to_369
- removed joint 474_to_373
- removed joint 475_to_373
- removed joint 476_to_373
- removed joint 478_to_377
- removed joint 479_to_377
- removed joint 480_to_377
- removed joint 48_to_37
- removed joint 49_to_37
- added joint 23_to_11: type revolute, parent 11, child 23, origin xyz=0.3410913428443227 0.9999 0.26632936129935403 rpy=9.553714901490551 3.4954292871862997 1.3277178800960172, axis 1 0 0, limit lower=3.1415 upper=-3.1415 effort=1 velocity=1
- joint 11_to_0: axis 0 0 1 -> 1 0 0; origin xyz=0.3487552547759922 0.4287697536007756 0.3870244515537885 rpy=6.266398357961349 5.646478324597923 2.9029606919443376 -> xyz=0.8024589819204132 0.9999 0.3153705944877665 rpy=6.558683593232514 3.138842939689139 3.0846537750239578
- joint 22_to_11: axis 0 0 1 -> 1 0 0; origin xyz=0.8704126844852472 0.15505226027397123 0.73850089972101 rpy=2.273734008552798 5.616259286488804 5.792622980579965 -> xyz=0.3410913428443227 0.9999 0.26632936129935403 rpy=6.369143267660368 3.4954292871862997 1.3277178800960172

Commit message: fix (kinda) issue where run_ga and realtime_from_csv fitness values differ

File: temp0.urdf (robot description, URDF)
Before this commit: robot pepe, 7 links, 6 joints
Links:
- removed link 15
- removed link 26
- link 0: mass 0.2993427185894939 -> 0.30020182443262416; geometry collision cylinder length=0.8202433794602948 radius=0.3413189181724402; visual cylinder length=0.8202433794602948 radius=0.3413189181724402
- link 11: mass 4.264862617044469 -> 0.38153612793751907; geometry collision cylinder length=0.4582811834682781 radius=0.5147861863462972; visual cylinder length=0.4582811834682781 radius=0.5147861863462972
- link 13: mass 4.264862617044469 -> 0.38153612793751907; geometry collision cylinder length=0.4582811834682781 radius=0.5147861863462972; visual cylinder length=0.4582811834682781 radius=0.5147861863462972
- link 22: mass 1.148510144550484 -> 1.3046278063617873; geometry collision cylinder length=0.4588754422273209 radius=0.9513076101344347; visual cylinder length=0.4588754422273209 radius=0.9513076101344347
- link 24: mass 1.148510144550484 -> 1.3046278063617873; geometry collision cylinder length=0.4588754422273209 radius=0.9513076101344347; visual cylinder length=0.4588754422273209 radius=0.9513076101344347
Joints:
- removed joint 15_to_0
- removed joint 26_to_15
- joint 11_to_0: origin xyz=0.30953915295501044 0.6895189303275684 0.5495245631995184 rpy=10.61683884527557 0.7206710599815701 6.282556988648868 -> xyz=0.9995893956930538 0.5762324414224341 0.03713008470708312 rpy=10.073548019933853 4.659504663191963 2.4836470791881746
- joint 13_to_0: origin xyz=0.30953915295501044 0.6895189303275684 0.5495245631995184 rpy=15.925258267913355 0.7206710599815701 6.282556988648868 -> xyz=0.9995893956930538 0.5762324414224341 0.03713008470708312 rpy=15.110322029900779 4.659504663191963 2.4836470791881746
- joint 22_to_11: origin xyz=0.25439540509300496 0.2289664483963053 0.13768350084241276 rpy=12.253927186812717 1.437516484625504 4.5765889171154335 -> xyz=0.06741544734933402 0.3974508836781886 0.8113373058363587 rpy=7.820595787783109 3.1197020396584545 1.1421056585581084
- joint 24_to_13: origin xyz=0.25439540509300496 0.2289664483963053 0.13768350084241276 rpy=12.253927186812717 1.437516484625504 4.5765889171154335 -> xyz=0.06741544734933402 0.3974508836781886 0.8113373058363587 rpy=7.820595787783109 3.1197020396584545 1.1421056585581084

File: test.urdf (robot description, URDF)
Before this commit: robot pepe, 4 links, 3 joints
Links:
- removed link 23
- added link 13, mass 0.21502869027662774; collision cylinder length=0.2582811834682781 radius=0.5147861863462972; visual cylinder length=0.2582811834682781 radius=0.5147861863462972
- added link 24, mass 1.3046278063617873; collision cylinder length=0.4588754422273209 radius=0.9513076101344347; visual cylinder length=0.4588754422273209 radius=0.9513076101344347
- link 0: mass 0.01063960190458224 -> 0.30020182443262416; geometry collision cylinder length=0.8202433794602948 radius=0.3413189181724402; visual cylinder length=0.8202433794602948 radius=0.3413189181724402
- link 11: mass 1.219129850958162 -> 0.21502869027662774; geometry collision cylinder length=0.2582811834682781 radius=0.5147861863462972; visual cylinder length=0.2582811834682781 radius=0.5147861863462972
- link 22: mass 0.01063960190458224 -> 1.3046278063617873; geometry collision cylinder length=0.4588754422273209 radius=0.9513076101344347; visual cylinder length=0.4588754422273209 radius=0.9513076101344347
Joints:
- removed joint 23_to_11
- added joint 13_to_0: type revolute, parent 0, child 13, origin xyz=0.9995893956930538 0.5762324414224341 0.03713008470708312 rpy=15.110322029900779 4.031186132474004 2.4836470791881746, axis 1 0 0, limit lower=3.1415 upper=-3.1415 effort=1 velocity=1
- added joint 24_to_13: type revolute, parent 13, child 24, origin xyz=0.06741544734933402 0.3974508836781886 0.8113373058363587 rpy=7.820595787783109 3.1197020396584545 1.1421056585581084, axis 0 1 0, limit lower=3.1415 upper=-3.1415 effort=1 velocity=1
- joint 11_to_0: origin xyz=0.8024589819204132 0.9999 0.3153705944877665 rpy=6.558683593232514 3.138842939689139 3.0846537750239578 -> xyz=0.9995893956930538 0.5762324414224341 0.03713008470708312 rpy=10.073548019933853 4.031186132474004 2.4836470791881746
- joint 22_to_11: axis 1 0 0 -> 0 1 0; origin xyz=0.3410913428443227 0.9999 0.26632936129935403 rpy=6.369143267660368 3.4954292871862997 1.3277178800960172 -> xyz=0.06741544734933402 0.3974508836781886 0.8113373058363587 rpy=7.820595787783109 3.1197020396584545 1.1421056585581084

Commit message: Am I overcomplicating fitness?

File: temp0.urdf (robot description, URDF)
Before this commit: robot pepe, 5 links, 4 joints
Links:
- added link 15, mass 0.24023544052366685; collision cylinder length=1.5622075801491697 radius=0.221245390702849; visual cylinder length=1.5622075801491697 radius=0.221245390702849
- added link 26, mass 2.387145400071626; collision cylinder length=1.9198692921114313 radius=0.6291130134070801; visual cylinder length=1.9198692921114313 radius=0.6291130134070801
- link 0: mass 0.30020182443262416 -> 0.1946704583259739; geometry collision cylinder length=0.27205881734562043 radius=0.4772475267572681; visual cylinder length=0.27205881734562043 radius=0.4772475267572681
- link 11: mass 0.38153612793751907 -> 0.24023544052366685; geometry collision cylinder length=1.5622075801491697 radius=0.221245390702849; visual cylinder length=1.5622075801491697 radius=0.221245390702849
- link 13: mass 0.38153612793751907 -> 0.24023544052366685; geometry collision cylinder length=1.5622075801491697 radius=0.221245390702849; visual cylinder length=1.5622075801491697 radius=0.221245390702849
- link 22: mass 1.3046278063617873 -> 2.387145400071626; geometry collision cylinder length=1.9198692921114313 radius=0.6291130134070801; visual cylinder length=1.9198692921114313 radius=0.6291130134070801
- link 24: mass 1.3046278063617873 -> 2.387145400071626; geometry collision cylinder length=1.9198692921114313 radius=0.6291130134070801; visual cylinder length=1.9198692921114313 radius=0.6291130134070801
Joints:
- added joint 15_to_0: type revolute, parent 0, child 15, origin xyz=0.013907691086566865 0.5897526669006181 0.0791590027893464 rpy=8.199481077757934 0.9768281932411039 5.502151616908443, axis 0 0 1, limit lower=3.1415 upper=-3.1415 effort=1 velocity=1
- added joint 26_to_15: type revolute, parent 15, child 26, origin xyz=0.2795887692477883 0.4131671429655013 0.3857780456794021 rpy=0.03831934115394378 0.41064288059501824 0.9690386488452966, axis 1 0 0, limit lower=3.1415 upper=-3.1415 effort=1 velocity=1
- joint 11_to_0: axis 1 0 0 -> 0 0 1; origin xyz=0.9995893956930538 0.5762324414224341 0.03713008470708312 rpy=10.073548019933853 4.659504663191963 2.4836470791881746 -> xyz=0.013907691086566865 0.5897526669006181 0.0791590027893464 rpy=4.099740538878967 0.9768281932411039 5.502151616908443
- joint 13_to_0: axis 1 0 0 -> 0 0 1; origin xyz=0.9995893956930538 0.5762324414224341 0.03713008470708312 rpy=15.110322029900779 4.659504663191963 2.4836470791881746 -> xyz=0.013907691086566865 0.5897526669006181 0.0791590027893464 rpy=6.14961080831845 0.9768281932411039 5.502151616908443
- joint 22_to_11: axis 0 1 0 -> 1 0 0; origin xyz=0.06741544734933402 0.3974508836781886 0.8113373058363587 rpy=7.820595787783109 3.1197020396584545 1.1421056585581084 -> xyz=0.2795887692477883 0.4131671429655013 0.3857780456794021 rpy=0.03831934115394378 0.41064288059501824 0.9690386488452966
- joint 24_to_13: axis 0 1 0 -> 1 0 0; origin xyz=0.06741544734933402 0.3974508836781886 0.8113373058363587 rpy=7.820595787783109 3.1197020396584545 1.1421056585581084 -> xyz=0.2795887692477883 0.4131671429655013 0.3857780456794021 rpy=0.03831934115394378 0.41064288059501824 0.9690386488452966

Commit message: rewrote fitness function with only 1 component
the sum of one over distance squared

File: temp0.urdf (robot description, URDF)
Before this commit: robot pepe, 7 links, 6 joints
Links:
- removed link 15
- removed link 22
- removed link 24
- removed link 26
- added link 12, mass 0.4969834148786758; collision cylinder length=0.5683753194119094 radius=0.5275679522764753; visual cylinder length=0.5683753194119094 radius=0.5275679522764753
- link 0: mass 0.1946704583259739 -> 0.11436015872527709; geometry collision cylinder length=1.2490119846959788 radius=0.17071792976729408; visual cylinder length=1.2490119846959788 radius=0.17071792976729408
- link 11: mass 0.24023544052366685 -> 0.4969834148786758; geometry collision cylinder length=0.5683753194119094 radius=0.5275679522764753; visual cylinder length=0.5683753194119094 radius=0.5275679522764753
- link 13: mass 0.24023544052366685 -> 0.4969834148786758; geometry collision cylinder length=0.5683753194119094 radius=0.5275679522764753; visual cylinder length=0.5683753194119094 radius=0.5275679522764753
Joints:
- removed joint 15_to_0
- removed joint 22_to_11
- removed joint 24_to_13
- removed joint 26_to_15
- added joint 12_to_0: type revolute, parent 0, child 12, origin xyz=0.19428614908922373 0.6224771454401942 0.3715902029451882 rpy=10.20994194127929 2.843485811118293 5.074191252773964, axis 0 1 0, limit lower=3.1415 upper=-3.1415 effort=1 velocity=1
- joint 11_to_0: axis 0 0 1 -> 0 1 0; origin xyz=0.013907691086566865 0.5897526669006181 0.0791590027893464 rpy=4.099740538878967 0.9768281932411039 5.502151616908443 -> xyz=0.19428614908922373 0.6224771454401942 0.3715902029451882 rpy=6.80662796085286 2.843485811118293 5.074191252773964
- joint 13_to_0: axis 0 0 1 -> 0 1 0; origin xyz=0.013907691086566865 0.5897526669006181 0.0791590027893464 rpy=6.14961080831845 0.9768281932411039 5.502151616908443 -> xyz=0.19428614908922373 0.6224771454401942 0.3715902029451882 rpy=13.61325592170572 2.843485811118293 5.074191252773964

File: test.urdf (robot description, URDF)
Before this commit: robot pepe, 5 links, 4 joints
Links:
- removed link 13
- removed link 22
- added link 12, mass 4.882347277368291; collision cylinder length=1.8777522670192015 radius=0.9097461990376425; visual cylinder length=1.8777522670192015 radius=0.9097461990376425
- added link 23, mass 0.12525409348090288; collision cylinder length=1.283128053011285 radius=0.17627309409780234; visual cylinder length=1.283128053011285 radius=0.17627309409780234
- link 0: mass 0.30020182443262416 -> 0.11603244283344977; geometry collision cylinder length=0.46410221704350696 radius=0.28210316579810013; visual cylinder length=0.46410221704350696 radius=0.28210316579810013
- link 11: mass 0.21502869027662774 -> 4.882347277368291; geometry collision cylinder length=1.8777522670192015 radius=0.9097461990376425; visual cylinder length=1.8777522670192015 radius=0.9097461990376425
- link 24: mass 1.3046278063617873 -> 0.12525409348090288; geometry collision cylinder length=1.283128053011285 radius=0.17627309409780234; visual cylinder length=1.283128053011285 radius=0.17627309409780234
Joints:
- removed joint 13_to_0
- removed joint 22_to_11
- removed joint 24_to_13
- added joint 12_to_0: type revolute, parent 0, child 12, origin xyz=0.4319144676027905 0.7709479173140095 0.7754871649637137 rpy=18.847670965946605 2.5108904133936685 2.9660927881855397, axis 0 1 0, limit lower=3.1415 upper=-3.1415 effort=1 velocity=1
- added joint 23_to_0: type revolute, parent 0, child 23, origin xyz=0.7216528522870539 0.5014602212875401 0.12678569535195694 rpy=15.911534068145672 1.4202069830539839 0.4839541055703547, axis 0 1 0, limit lower=3.1415 upper=-3.1415 effort=1 velocity=1
- added joint 24_to_0: type revolute, parent 0, child 24, origin xyz=0.7216528522870539 0.5014602212875401 0.12678569535195694 rpy=19.88941758518209 1.4202069830539839 0.4839541055703547, axis 0 1 0, limit lower=3.1415 upper=-3.1415 effort=1 velocity=1
- joint 11_to_0: axis 1 0 0 -> 0 1 0; origin xyz=0.9995893956930538 0.5762324414224341 0.03713008470708312 rpy=10.073548019933853 4.031186132474004 2.4836470791881746 -> xyz=0.4319144676027905 0.7709479173140095 0.7754871649637137 rpy=12.565113977297736 2.5108904133936685 2.9660927881855397
